File: astro-medallion.kicad_pcb (KiCad board)
At the start: 2 copper layers, 149.3 x 149.3 mm, 203 parts, among them U1 74HC595, U10 74LS540, U11 ESP32-C3-DevKitM-1, U12 MCP7940N-xSN, U2 74HC595, U3 74HC595, U4 74HC595, U5 74HC595, U6 74LS540, U7 74LS540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

Commit message: reversed the labels of the signs to increase counter-clockwise
Parts:
- moved G*** 133.2 mm to (51.4, 97.6), turned to 90 degrees
- moved G*** 133.2 mm to (184.6, 97.6), turned to -90 degrees
- moved G*** 115.4 mm to (175.7, 64.4), turned to -60 degrees
- moved G*** 115.4 mm to (60.3, 64.3), turned to 60 degrees
- moved G*** 115.4 mm to (60.3, 130.9), turned to 120 degrees
- moved G*** 115.4 mm to (175.7, 130.9), turned to -120 degrees
- moved G*** 66.6 mm to (151.3, 40.0), turned to -30 degrees
- moved G*** 66.6 mm to (84.7, 39.9), turned to 30 degrees
- moved G*** 66.6 mm to (151.3, 155.4), turned to -150 degrees
- moved G*** 66.6 mm to (84.7, 155.4), turned to 150 degrees
